Commit message: Updated URDF models.

File: pioneer_description/urdf/pioneer3dx.xacro (robot description, xacro)
@@ -25,5 +25,6 @@
 			<origin xyz="0 0 0" rpy="0 0 0"/>
 			<geometry>
-				<box size="0.43 0.277 0.17"/>
+				<mesh filename="package://pioneer_description/meshes/p3dx_meshes/chassis.stl"/>
+				<!--box size="0.43 0.277 0.17"/-->
 			</geometry>
 		</collision>
@@ -60,5 +61,6 @@
 			<origin xyz="0 0 0" rpy="0 0 0"/>
 			<geometry>
-				<box size="0.44 0.38 0.005"/>
+				<mesh filename="package://pioneer_description/meshes/p3dx_meshes/top.stl"/>
+				<!--box size="0.44 0.38 0.005"/-->
 			</geometry>
 		</collision>
@@ -91,5 +93,5 @@
 		  <origin xyz="0 0 0" rpy="0 0 0"/>
 		  <geometry>
-			  <box size="0 0 0"/>
+			  <mesh filename="package://pioneer_description/meshes/p3dx_meshes/swivel.stl"/>
 		  </geometry>
 	  </collision>
@@ -113,5 +115,5 @@
 		  <origin xyz="0 0 0" rpy="0 0 0"/>
 		  <geometry>
-			  <box size="0 0 0"/>
+			  <mesh filename="package://pioneer_description/meshes/p3dx_meshes/center_hubcap.stl"/>
 		  </geometry>
 	  </collision>
@@ -141,7 +143,8 @@
 	  </visual>
 	  <collision>
-		  <origin xyz="0 0 0" rpy="${-3.1415927/2.0} 0 0"/>
+		  <origin xyz="0 0 0" rpy="0 0 0"/>
 		  <geometry>
-			  <cylinder radius="0.0375" length="0.03"/>
+		    <mesh filename="package://pioneer_description/meshes/p3dx_meshes/center_wheel.stl"/>
+			  <!--<cylinder radius="0.0375" length="0.03"/>-->
 		  </geometry>
 	  </collision>
@@ -177,7 +180,8 @@
 		</visual>
 		<collision>
-			<origin xyz="0 0 0" rpy="${-3.1415927/2.0} 0 0"/>
-			<geometry>
-				<cylinder radius="0.092" length="0.04"/>
+			<origin xyz="0 0 0" rpy="0 0 0"/>
+			<geometry>
+			  <mesh filename="package://pioneer_description/meshes/p3dx_meshes/left_wheel.stl"/>
+				<!--<cylinder radius="0.092" length="0.04"/>-->
 			</geometry>
 		</collision>
@@ -199,5 +203,5 @@
 			<origin xyz="0 0 0" rpy="0 0 0"/>
 			<geometry>
-				<box size="0 0 0"/>
+				<mesh filename="package://pioneer_description/meshes/p3dx_meshes/left_hubcap.stl"/>
 			</geometry>
 		</collision>
@@ -228,7 +232,8 @@
 		</visual>
 		<collision>
-			<origin xyz="0 0 0" rpy="${-3.1415927/2.0} 0 0"/>
-			<geometry>
-				<cylinder radius="0.092" length="0.04"/>
+			<origin xyz="0 0 0" rpy="0 0 0"/>
+			<geometry>
+			  <mesh filename="package://pioneer_description/meshes/p3dx_meshes/right_wheel.stl"/>
+				<!--<cylinder radius="0.092" length="0.04"/>-->
 			</geometry>
 		</collision>
@@ -250,5 +255,5 @@
 			<origin xyz="0 0 0" rpy="0 0 0"/>
 			<geometry>
-				<box size="0 0 0"/>
+				<mesh filename="package://pioneer_description/meshes/p3dx_meshes/right_hubcap.stl"/>
 			</geometry>
 		</collision>
@@ -272,5 +277,5 @@
 			<origin xyz="0 0 0" rpy="0 0 0"/>
 			<geometry>
-				<box size="0 0 0"/>
+				<mesh filename="package://pioneer_description/meshes/p3dx_meshes/front_sonar.stl"/>
 			</geometry>
 		</collision>
@@ -298,5 +303,5 @@
 			<origin xyz="0 0 0" rpy="0 0 0"/>
 			<geometry>
-				<box size="0 0 0"/>
+				<mesh filename="package://pioneer_description/meshes/p3dx_meshes/back_sonar.stl"/>
 			</geometry>
 		</collision>
@@ -311,5 +316,5 @@
     <parent link="camera_link"/>
     <child link="hokuyo_link"/>
-  </joint>-->
+  </joint>
   <!-- Hokuyo Laser -->
   <link name="hokuyo_link">
@@ -317,5 +322,6 @@
       <origin xyz="0 0 0" rpy="0 0 0"/>
       <geometry>
-	      <box size="0.05 0.05 0.071"/>
+        <mesh filename="package://pioneer_description/meshes/hokuyo.dae"/>
+	      <!--box size="0.05 0.05 0.071"/-->
       </geometry>
     </collision>

Commit message: Updated gazebo model hokuyo link name to 'laser', standardise across hardware and software experiments

File: pioneer_description/urdf/pioneer3dx.xacro (robot description, xacro)
@@ -315,8 +315,8 @@
     <origin xyz="0 0 0.085" rpy="0 0 0"/>
     <parent link="camera_link"/>
-    <child link="hokuyo_link"/>
+    <child link="laser"/>
   </joint>
   <!-- Hokuyo Laser -->
-  <link name="hokuyo_link">
+  <link name="laser">
     <collision>
       <origin xyz="0 0 0" rpy="0 0 0"/>
